Commit message: Chassis robot, simulation of walking and camera movement

File: urdf/fobo2.urdf (robot description, URDF)
Before this commit: robot fobo2, 9 links, 8 joints
Links:
- link stick-back: geometry collision cylinder length=0.2654 radius=0.015; visual cylinder length=0.2654 radius=0.015
- link stick-front: geometry collision cylinder length=0.2654 radius=0.015; visual cylinder length=0.2654 radius=0.015
Joints:
- joint ball-back-joint: origin xyz=0 0 -0.13275 rpy=0 0 0 -> xyz={-(chassis_length/2 - stick_offset)} 0 -0.26 rpy=0 0 0; parent stick-back -> base_link
- joint ball-front-joint: origin xyz=0 0 -0.13275 rpy=0 0 0 -> xyz=0.22500000000000003 0 -0.26 rpy=0 0 0; parent stick-front -> base_link
- joint stick-back-base: origin xyz=-0.22500000000000003 0 -0.13275 rpy=0 0 0 -> xyz=-0.22500000000000003 0 -0.1327 rpy=0 0 0
- joint stick-front-base: origin xyz=0.22500000000000003 0 -0.13275 rpy=0 0 0 -> xyz=0.22500000000000003 0 -0.1327 rpy=0 0 0

File: urdf/fobo2.xacro (robot description, xacro)
@@ -22,5 +22,5 @@
     <xacro:property name="stick_mass" value="0.015"/>
     <!-- Stick length can't be automatically calculated -->
-    <xacro:property name="stick_length" value="0.2655" />
+    <xacro:property name="stick_length" value="0.2654" />
     <!-- define colors -->
     <material name="white">
@@ -164,5 +164,5 @@
     <xacro:static_joint name="stick-front-base" parent="base_link" child="stick-front" xyz="${chassis_length/2 - stick_offset} 0 ${-stick_length/2}" rpy="0 0 0" />
     <xacro:static_joint name="stick-back-base" parent="base_link" child="stick-back" xyz="${-(chassis_length/2 - stick_offset)} 0 ${-stick_length/2}" rpy="0 0 0" />
-    <xacro:sphere_joint name="ball-front-joint" parent="stick-front" child="ball-front" xyz="0 0 ${-stick_length/2}" />
-    <xacro:sphere_joint name="ball-back-joint" parent="stick-back" child="ball-back" xyz="0 0 ${-stick_length/2}" />
+    <xacro:sphere_joint name="ball-front-joint" parent="base_link" child="ball-front" xyz="${chassis_length/2 - stick_offset} 0 ${-chassis_depth/2 - wheel_radius + ball_radius}" />
+    <xacro:sphere_joint name="ball-back-joint" parent="base_link" child="ball-back" xyz="{-(chassis_length/2 - stick_offset)} 0 ${-chassis_depth/2 - wheel_radius + ball_radius}" />
 </robot>

Commit message: Change urdf model and add optuna optimization hyperparams

File: urdf/fobo2.urdf (robot description, URDF)
Before this commit: robot fobo2, 9 links, 8 joints
Links:
- link base_link: mass 1 -> 0.654
Joints:
- joint ball-back-joint: axis (none) -> 0 0 1; type floating -> spherical
- joint ball-front-joint: axis (none) -> 0 0 1; type floating -> spherical

File: urdf/fobo2.xacro (robot description, xacro)
@@ -5,5 +5,5 @@
     <xacro:property name="chassis_width" value="0.35"/>
     <xacro:property name="chassis_depth" value="0.01"/>
-    <xacro:property name="chassis_mass" value="1"/>
+    <xacro:property name="chassis_mass" value="0.654"/>
     <!-- Motor cylinder parameters -->
     <xacro:property name="motor_radius" value="0.032"/>
@@ -135,9 +135,9 @@
     </xacro:macro>
     <xacro:macro name="sphere_joint" params="name parent child xyz">
-        <joint name="${name}" type="floating">
+        <joint name="${name}" type="spherical">
             <parent link="${parent}" />
             <child link="${child}" />
             <origin xyz="${xyz}" rpy="0 0 0"/>
-            <!-- <axis xyz="0 0 1"/>  -->
+            <axis xyz="0 0 1"/>
         </joint>
     </xacro:macro>
