Commit message: Add more realistic representation of real robot

File: fobo2_env/fobo2_env/src/models/fobo2.urdf (robot description, URDF)
Before this commit: robot fobo2, 9 links, 8 joints
Links:
- link ball-back: geometry collision sphere radius=0.03; visual sphere radius=0.03
- link ball-front: geometry collision sphere radius=0.03; visual sphere radius=0.03
- link base_link: geometry collision box size=0.55 0.35 0.01; visual box size=0.55 0.35 0.01
- link motor-left: geometry collision cylinder length=0.105 radius=0.032; visual cylinder length=0.105 radius=0.032
- link motor-right: geometry collision cylinder length=0.105 radius=0.032; visual cylinder length=0.105 radius=0.032
- link stick-back: geometry collision cylinder length=0.102 radius=0.015; visual cylinder length=0.102 radius=0.015
- link stick-front: geometry collision cylinder length=0.102 radius=0.015; visual cylinder length=0.102 radius=0.015
- link wheel-left: geometry collision cylinder length=0.088 radius=0.12; visual cylinder length=0.088 radius=0.12
- link wheel-right: geometry collision cylinder length=0.088 radius=0.12; visual cylinder length=0.088 radius=0.12
Joints:
- joint ball-back-joint: origin xyz={-(chassis_length/2 - stick_offset)} 0 -0.26 rpy=0 0 0 -> xyz=-0.22500000000000003 0 -0.115 rpy=0 0 0
- joint ball-front-joint: origin xyz=0.22500000000000003 0 -0.26 rpy=0 0 0 -> xyz=0.22500000000000003 0 -0.115 rpy=0 0 0
- joint motor-left-base: origin xyz=0 -0.034999999999999996 -0.055 rpy=0 1.5707 1.5707 -> xyz=0 -0.1325 -0.026000000000000002 rpy=0 1.5707 1.5707
- joint motor-right-base: origin xyz=0 0.034999999999999996 -0.055 rpy=0 1.5707 1.5707 -> xyz=0 0.1325 -0.026000000000000002 rpy=0 1.5707 1.5707
- joint stick-back-base: origin xyz=-0.22500000000000003 0 -0.1327 rpy=0 0 0 -> xyz=-0.22500000000000003 0 -0.051 rpy=0 0 0
- joint stick-front-base: origin xyz=0.22500000000000003 0 -0.1327 rpy=0 0 0 -> xyz=0.22500000000000003 0 -0.051 rpy=0 0 0
- joint wheel-motor-left: origin xyz=0 0 -0.2 rpy=0 0 0 -> xyz=0 0 -0.0965 rpy=0 0 0
- joint wheel-motor-right: origin xyz=0 0 0.2 rpy=0 0 0 -> xyz=0 0 0.0965 rpy=0 0 0

File: fobo2_env/fobo2_env/src/models/wall.urdf (robot description, URDF)
Before this commit: robot box, 1 links, 0 joints
Links:
- link box: geometry collision box size=6 40 0.2; visual box size=6 40 0.2

File: urdf/fobo2.urdf (robot description, URDF)
Before this commit: robot fobo2, 9 links, 8 joints
Links:
- link ball-back: geometry collision sphere radius=0.03; visual sphere radius=0.03
- link ball-front: geometry collision sphere radius=0.03; visual sphere radius=0.03
- link base_link: geometry collision box size=0.55 0.35 0.01; visual box size=0.55 0.35 0.01
- link motor-left: mass 1 -> 0.438; geometry collision cylinder length=0.105 radius=0.032; visual cylinder length=0.105 radius=0.032
- link motor-right: mass 1 -> 0.438; geometry collision cylinder length=0.105 radius=0.032; visual cylinder length=0.105 radius=0.032
- link stick-back: geometry collision cylinder length=0.102 radius=0.015; visual cylinder length=0.102 radius=0.015
- link stick-front: geometry collision cylinder length=0.102 radius=0.015; visual cylinder length=0.102 radius=0.015
- link wheel-left: mass 1 -> 0.237; geometry collision cylinder length=0.088 radius=0.12; visual cylinder length=0.088 radius=0.12
- link wheel-right: mass 1 -> 0.237; geometry collision cylinder length=0.088 radius=0.12; visual cylinder length=0.088 radius=0.12
Joints:
- joint ball-back-joint: origin xyz={-(chassis_length/2 - stick_offset)} 0 -0.26 rpy=0 0 0 -> xyz=-0.22500000000000003 0 -0.115 rpy=0 0 0
- joint ball-front-joint: origin xyz=0.22500000000000003 0 -0.26 rpy=0 0 0 -> xyz=0.22500000000000003 0 -0.115 rpy=0 0 0
- joint motor-left-base: origin xyz=0 -0.034999999999999996 -0.055 rpy=0 1.5707 1.5707 -> xyz=0 -0.1325 -0.026000000000000002 rpy=0 1.5707 1.5707
- joint motor-right-base: origin xyz=0 0.034999999999999996 -0.055 rpy=0 1.5707 1.5707 -> xyz=0 0.1325 -0.026000000000000002 rpy=0 1.5707 1.5707
- joint stick-back-base: origin xyz=-0.22500000000000003 0 -0.1327 rpy=0 0 0 -> xyz=-0.22500000000000003 0 -0.051 rpy=0 0 0
- joint stick-front-base: origin xyz=0.22500000000000003 0 -0.1327 rpy=0 0 0 -> xyz=0.22500000000000003 0 -0.051 rpy=0 0 0
- joint wheel-motor-left: origin xyz=0 0 -0.2 rpy=0 0 0 -> xyz=0 0 -0.0965 rpy=0 0 0
- joint wheel-motor-right: origin xyz=0 0 0.2 rpy=0 0 0 -> xyz=0 0 0.0965 rpy=0 0 0

File: urdf/fobo2.xacro (robot description, xacro)
@@ -4,17 +4,17 @@
     <xacro:property name="chassis_length" value="0.55"/>
     <xacro:property name="chassis_width" value="0.35"/>
-    <xacro:property name="chassis_depth" value="0.1"/>
+    <xacro:property name="chassis_depth" value="0.01"/>
     <xacro:property name="chassis_mass" value="1"/>
     <!-- Motor cylinder parameters -->
-    <xacro:property name="motor_radius" value="0.01"/>
-    <xacro:property name="motor_length" value="0.3"/>
-    <xacro:property name="motor_mass" value="1"/>
+    <xacro:property name="motor_radius" value="0.032"/>
+    <xacro:property name="motor_length" value="0.105"/>
+    <xacro:property name="motor_mass" value="0.438"/>
     <xacro:property name="motor_offset" value="0.01"/>
     <!-- wheel parameters -->
-    <xacro:property name="wheel_radius" value="0.225"/>
-    <xacro:property name="wheel_length" value="0.1"/>
-    <xacro:property name="wheel_mass" value="1"/>
+    <xacro:property name="wheel_radius" value="0.12"/>
+    <xacro:property name="wheel_length" value="0.088"/>
+    <xacro:property name="wheel_mass" value="0.237"/>
     <!-- Ball parameters -->
-    <xacro:property name="ball_radius" value="0.015"/>
+    <xacro:property name="ball_radius" value="0.030"/>
     <xacro:property name="ball_mass" value="1"/>
     <xacro:property name="stick_offset" value="0.05"/>
@@ -22,5 +22,5 @@
     <xacro:property name="stick_mass" value="0.015"/>
     <!-- Stick length can't be automatically calculated -->
-    <xacro:property name="stick_length" value="0.2654" />
+    <xacro:property name="stick_length" value="0.102" />
     <!-- define colors -->
     <material name="white">
@@ -156,6 +156,6 @@
     <xacro:sphere_link link_name="ball-back" radius="${ball_radius}" mass="${ball_mass}" color="red" />
     <!-- Motor joints -->
-    <xacro:static_joint name="motor-right-base" parent="base_link" child="motor-right" xyz="0 ${chassis_width/2 - motor_length/2  + motor_offset} ${-(chassis_depth/2 + motor_radius/2)}" rpy="0 1.5707 1.5707"/>
-    <xacro:static_joint name="motor-left-base" parent="base_link" child="motor-left" xyz="0 ${-(chassis_width/2 - motor_length/2 + motor_offset)} ${-(chassis_depth/2 + motor_radius/2)}" rpy="0 1.5707 1.5707"/>
+    <xacro:static_joint name="motor-right-base" parent="base_link" child="motor-right" xyz="0 ${chassis_width/2 - motor_length/2  + motor_offset} ${-(chassis_depth + motor_radius/2)}" rpy="0 1.5707 1.5707"/>
+    <xacro:static_joint name="motor-left-base" parent="base_link" child="motor-left" xyz="0 ${-(chassis_width/2 - motor_length/2 + motor_offset)} ${-(chassis_depth + motor_radius/2)}" rpy="0 1.5707 1.5707"/>
     <!-- Wheel joints -->
     <xacro:wheel_joint name="wheel-motor-right" parent="motor-right" child="wheel-right" xyz="0 0 ${motor_length/2 + wheel_length/2}"/>
@@ -163,6 +163,6 @@
     <!-- Ball joints -->
     <xacro:static_joint name="stick-front-base" parent="base_link" child="stick-front" xyz="${chassis_length/2 - stick_offset} 0 ${-stick_length/2}" rpy="0 0 0" />
-    <xacro:static_joint name="stick-back-base" parent="base_link" child="stick-back" xyz="${-(chassis_length/2 - stick_offset)} 0 ${-stick_length/2}" rpy="0 0 0" />
-    <xacro:sphere_joint name="ball-front-joint" parent="base_link" child="ball-front" xyz="${chassis_length/2 - stick_offset} 0 ${-chassis_depth/2 - wheel_radius + ball_radius}" />
-    <xacro:sphere_joint name="ball-back-joint" parent="base_link" child="ball-back" xyz="{-(chassis_length/2 - stick_offset)} 0 ${-chassis_depth/2 - wheel_radius + ball_radius}" />
+    <xacro:static_joint name="stick-back-base" parent="base_link" child="stick-back" xyz="${-(chassis_length/2 - stick_offset)} 0 ${-stick_length/2s}" rpy="0 0 0" />
+    <xacro:sphere_joint name="ball-front-joint" parent="base_link" child="ball-front" xyz="${chassis_length/2 - stick_offset} 0 ${-chassis_depth - wheel_radius + ball_radius/2}" />
+    <xacro:sphere_joint name="ball-back-joint" parent="base_link" child="ball-back" xyz="${-(chassis_length/2 - stick_offset)} 0 ${-chassis_depth - wheel_radius + ball_radius/2}" />
 </robot>

Commit message: Add input normalization and correct depth buffer memory

File: fobo2_env/fobo2_env/src/models/fobo2.urdf (robot description, URDF)
Before this commit: robot fobo2, 9 links, 8 joints
Links:
- link base_link: mass 1 -> 0.654
- link motor-left: mass 1 -> 0.438
- link motor-right: mass 1 -> 0.438
- link wheel-left: mass 1 -> 0.237
- link wheel-right: mass 1 -> 0.237
Joints:
- joint ball-back-joint: axis (none) -> 0 0 1; type floating -> spherical
- joint ball-front-joint: axis (none) -> 0 0 1; type floating -> spherical

Commit message: Delete useless meshes, update requirements, Add train_fobo and train optuna functional code, Correct action scaling

File: fobo2_env/fobo2_env/src/models/fobo2.urdf (robot description, URDF)
Before this commit: robot fobo2, 9 links, 8 joints
Joints:
- joint stick-back-base: origin xyz=-0.22500000000000003 0 -0.051 rpy=0 0 0 -> xyz=0.22500000000000003 0 -0.051 rpy=0 0 0
- joint stick-front-base: origin xyz=0.22500000000000003 0 -0.051 rpy=0 0 0 -> xyz=-0.22500000000000003 0 -0.051 rpy=0 0 0
- joint wheel-motor-left: axis 0 0 1 -> 0 0 -1
- joint wheel-motor-right: axis 0 0 1 -> 0 0 -1

File: urdf/fobo2.xacro (robot description, xacro)
@@ -23,5 +23,5 @@
     <!-- Stick length can't be automatically calculated -->
     <xacro:property name="stick_length" value="0.102" />
-    <!-- define colors -->
+    <!-- Define colors -->
     <material name="white">
         <color rgba="1 1 1 1"/>
@@ -32,4 +32,7 @@
     <material name="red">
         <color rgba="1 0 0 1"/>
+    </material>
+    <material name="blue">
+        <color rgba="0 0 1 1"/>
     </material>
     <xacro:macro name="cylinder_inertia" params="m r h">
@@ -56,7 +59,5 @@
             </geometry>
                 <origin rpy="0 0 0" xyz="0 0 0"/>
-                <material name="${color}">
-                    <!-- <color rgba="1 1 1 1"/> -->
-                </material>
+                <material name="${color}"/>
             </visual>
             <collision>
@@ -72,27 +73,33 @@
         </link>
     </xacro:macro>
-    <xacro:macro name="cylinder_link" params="link_name radius length mass color">
-        <link name="${link_name}">
-            <visual>
-                <geometry>
-                    <cylinder radius="${radius}" length="${length}"/>
-                </geometry>
-                <origin rpy="0 0 0" xyz="0 0 0"/>
-                <material name="${color}">
-                    <color rgba="1 1 1 1"/>
-                </material>
-            </visual>
-            <collision>
-                <geometry>
-                    <cylinder radius="${radius}" length="${length}"/>
-                </geometry>
-                <origin rpy="0 0 0" xyz="0 0 0"/>
-            </collision>
-            <inertial>
-                <mass value="${mass}"/>
-                <xacro:cylinder_inertia m="${mass}" r="${radius}" h="${length}" />
-            </inertial>
-        </link>
-    </xacro:macro>
+<xacro:macro name="cylinder_link" params="link_name radius length mass color lateral_friction">
+    <link name="${link_name}">
+        <visual>
+            <geometry>
+                <cylinder radius="${radius}" length="${length}"/>
+            </geometry>
+            <origin rpy="0 0 0" xyz="0 0 0"/>
+            <material name="${color}"/>
+        </visual>
+        <collision>
+            <geometry>
+                <cylinder radius="${radius}" length="${length}"/>
+            </geometry>
+            <origin rpy="0 0 0" xyz="0 0 0"/>
+            <surface>
+                <friction>
+                    <ode>
+                        <mu>${lateral_friction}</mu>
+                        <mu2>${lateral_friction}</mu2>
+                    </ode>
+                </friction>
+            </surface>
+        </collision>
+        <inertial>
+            <mass value="${mass}"/>
+            <xacro:cylinder_inertia m="${mass}" r="${radius}" h="${length}" />
+        </inertial>
+    </link>
+</xacro:macro>
     <xacro:macro name="sphere_link" params="link_name radius mass color">
         <link name="${link_name}">
@@ -102,7 +109,5 @@
                 </geometry>
                 <origin rpy="0 0 0" xyz="0 0 0"/>
-                <material name="${color}">
-                    <color rgba="1 1 1 1"/>
-                </material>
+                <material name="${color}"/>
             </visual>
             <collision>
@@ -131,5 +136,5 @@
             <child link="${child}" />
             <origin xyz="${xyz}" rpy="0 0 0"/>
-            <axis xyz="0 0 1"/>
+            <axis xyz="0 0 -1"/>
         </joint>
     </xacro:macro>
@@ -145,12 +150,12 @@
     <xacro:box_link link_name="base_link" length="${chassis_length}" width="${chassis_width}" depth="${chassis_depth}" mass="${chassis_mass}" color="white" />
     <!-- Motor links -->
-    <xacro:cylinder_link link_name="motor-right" radius="${motor_radius}" length="${motor_length}" mass="${motor_mass}" color="white" />
-    <xacro:cylinder_link link_name="motor-left" radius="${motor_radius}" length="${motor_length}" mass="${motor_mass}" color="white" />
+    <xacro:cylinder_link link_name="motor-right" radius="${motor_radius}" length="${motor_length}" mass="${motor_mass}" color="white" lateral_friction="0" />
+    <xacro:cylinder_link link_name="motor-left" radius="${motor_radius}" length="${motor_length}" mass="${motor_mass}" color="white" lateral_friction="0" />
     <!-- Wheel links -->
-    <xacro:cylinder_link link_name="wheel-right" radius="${wheel_radius}" length="${wheel_length}" mass="${wheel_mass}" color="black" />
-    <xacro:cylinder_link link_name="wheel-left" radius="${wheel_radius}" length="${wheel_length}" mass="${wheel_mass}" color="black" />
+    <xacro:cylinder_link link_name="wheel-right" radius="${wheel_radius}" length="${wheel_length}" mass="${wheel_mass}" color="black" lateral_friction="1.0" />
+    <xacro:cylinder_link link_name="wheel-left" radius="${wheel_radius}" length="${wheel_length}" mass="${wheel_mass}" color="black" lateral_friction="1.0" />
     <!-- Ball links -->
-    <xacro:cylinder_link link_name="stick-front" radius="${stick_radius}" length="${stick_length}" mass="${stick_mass}" color="black" />
-    <xacro:cylinder_link link_name="stick-back" radius="${stick_radius}" length="${stick_length}" mass="${stick_mass}" color="black" />
+    <xacro:cylinder_link link_name="stick-front" radius="${stick_radius}" length="${stick_length}" mass="${stick_mass}" color="blue" lateral_friction="0" />
+    <xacro:cylinder_link link_name="stick-back" radius="${stick_radius}" length="${stick_length}" mass="${stick_mass}" color="black" lateral_friction="0" />
     <xacro:sphere_link link_name="ball-front" radius="${ball_radius}" mass="${ball_mass}" color="red" />
     <xacro:sphere_link link_name="ball-back" radius="${ball_radius}" mass="${ball_mass}" color="red" />
@@ -162,6 +167,6 @@
     <xacro:wheel_joint name="wheel-motor-left" parent="motor-left" child="wheel-left" xyz="0 0 ${-(motor_length/2 + wheel_length/2)}"/>
     <!-- Ball joints -->
-    <xacro:static_joint name="stick-front-base" parent="base_link" child="stick-front" xyz="${chassis_length/2 - stick_offset} 0 ${-stick_length/2}" rpy="0 0 0" />
-    <xacro:static_joint name="stick-back-base" parent="base_link" child="stick-back" xyz="${-(chassis_length/2 - stick_offset)} 0 ${-stick_length/2s}" rpy="0 0 0" />
+    <xacro:static_joint name="stick-back-base" parent="base_link" child="stick-back" xyz="${chassis_length/2 - stick_offset} 0 ${-stick_length/2}" rpy="0 0 0" />
+    <xacro:static_joint name="stick-front-base" parent="base_link" child="stick-front" xyz="${-(chassis_length/2 - stick_offset)} 0 ${-stick_length/2s}" rpy="0 0 0" />
     <xacro:sphere_joint name="ball-front-joint" parent="base_link" child="ball-front" xyz="${chassis_length/2 - stick_offset} 0 ${-chassis_depth - wheel_radius + ball_radius/2}" />
     <xacro:sphere_joint name="ball-back-joint" parent="base_link" child="ball-back" xyz="${-(chassis_length/2 - stick_offset)} 0 ${-chassis_depth - wheel_radius + ball_radius/2}" />
